File: elec/connected_garden_pcb/connected_garden_pcb.sch (KiCad schematic (older format))
At the start: 21 parts, among them J1 Moisture1, J2 Moisture2, J3 Moisture3, J4 Moisture4, J5 Moisture5, SW1 Reset, SW2 Flash, U1 TP4056-18650, U2 MCP3208, U3 SPX3819M5-L-3-3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

Commit message: [Elec] Updates project lib with TP4056-18650
Parts:
- C1: footprint (none) -> Capacitor_THT:C_Radial_D6.3mm_H7.0mm_P2.50mm
- J1, J2, J3, J4, J5: footprint (none) -> Connector_PinHeader_2.54mm:PinHeader_1x03_P2.54mm_Vertical
- J6: renamed from J?; footprint (none) -> TerminalBlock_RND:TerminalBlock_RND_205-00001_1x02_P5.00mm_Horizontal
- J7: renamed from J?; value Conn_01x03_Female -> UART out; footprint (none) -> Connector_PinHeader_2.54mm:PinHeader_1x03_P2.54mm_Vertical
- R1, R2, R3, R4, R5: footprint (none) -> Resistor_THT:R_Axial_DIN0207_L6.3mm_D2.5mm_P10.16mm_Horizontal
- R6: renamed from R?; footprint (none) -> Resistor_THT:R_Axial_DIN0207_L6.3mm_D2.5mm_P10.16mm_Horizontal
- SW1, SW2: footprint (none) -> Button_Switch_THT:SW_TH_Tactile_Omron_B3F-10xx
- U1: footprint (none) -> connected_garden_footprints:TP4056-18650
- U2: footprint (none) -> Package_DIP:DIP-16_W7.62mm_Socket_LongPads
- U4: footprint (none) -> Connector_PinSocket_2.54mm:PinSocket_1x04_P2.54mm_Vertical
Changed lines of the file:
@@
 Comment4 ""
 $EndDescr
-$Comp
-L connected_garden_lib:TP4056-18650 U1
-U 1 1 5D27D33C
-P 1500 1150
-F 0 "U1" H 1475 1625 50  0000 C CNN
-F 1 "TP4056-18650" H 1475 1534 50  0000 C CNN
-F 2 "" H 1450 1150 50  0001 C CNN
-F 3 "" H 1450 1150 50  0001 C CNN
-	1    1500 1150
-	1    0    0    -1
-$EndComp
 Wire Wire Line
 	8150 3950 8150 4100
@@
 F 0 "U4" H 5920 1446 50  0000 R CNN
 F 1 "DHT11" H 5920 1355 50  0000 R CNN
-F 2 "" H 6300 1650 50  0001 C CNN
+F 2 "Connector_PinSocket_2.54mm:PinSocket_1x04_P2.54mm_Vertical" H 6300 1650 50  0001 C CNN
 F 3 "http://akizukidenshi.com/download/ds/aosong/DHT11.pdf" H 6300 1650 50  0001 C CNN
 	1    6150 1400
@@
 F 0 "U2" H 1700 5828 50  0000 C CNN
 F 1 "MCP3208" H 1700 5737 50  0000 C CNN
-F 2 "" H 1800 5250 50  0001 C CNN
+F 2 "Package_DIP:DIP-16_W7.62mm_Socket_LongPads" H 1800 5250 50  0001 C CNN
 F 3 "http://ww1.microchip.com/downloads/en/DeviceDoc/21298c.pdf" H 1800 5250 50  0001 C CNN
 	1    1700 5150
@@
 F 0 "C1" H 3765 1296 50  0000 L CNN
 F 1 "1µF" H 3765 1205 50  0000 L CNN
-F 2 "" H 3688 1100 50  0001 C CNN
+F 2 "Capacitor_THT:C_Radial_D6.3mm_H7.0mm_P2.50mm" H 3688 1100 50  0001 C CNN
 F 3 "~" H 3650 1250 50  0001 C CNN
 	1    3650 1250
@@
 F 0 "J1" H 3927 4576 50  0000 L CNN
 F 1 "Moisture1" H 3927 4485 50  0000 L CNN
-F 2 "" H 3900 4550 50  0001 C CNN
+F 2 "Connector_PinHeader_2.54mm:PinHeader_1x03_P2.54mm_Vertical" H 3900 4550 50  0001 C CNN
 F 3 "~" H 3900 4550 50  0001 C CNN
 	1    3900 4550
@@
 F 0 "J2" H 3927 4926 50  0000 L CNN
 F 1 "Moisture2" H 3927 4835 50  0000 L CNN
-F 2 "" H 3900 4900 50  0001 C CNN
+F 2 "Connector_PinHeader_2.54mm:PinHeader_1x03_P2.54mm_Vertical" H 3900 4900 50  0001 C CNN
 F 3 "~" H 3900 4900 50  0001 C CNN
 	1    3900 4900
@@
 F 0 "J3" H 3927 5276 50  0000 L CNN
 F 1 "Moisture3" H 3927 5185 50  0000 L CNN
-F 2 "" H 3900 5250 50  0001 C CNN
+F 2 "Connector_PinHeader_2.54mm:PinHeader_1x03_P2.54mm_Vertical" H 3900 5250 50  0001 C CNN
 F 3 "~" H 3900 5250 50  0001 C CNN
 	1    3900 5250
@@
 F 0 "J4" H 3927 5626 50  0000 L CNN
 F 1 "Moisture4" H 3927 5535 50  0000 L CNN
-F 2 "" H 3900 5600 50  0001 C CNN
+F 2 "Connector_PinHeader_2.54mm:PinHeader_1x03_P2.54mm_Vertical" H 3900 5600 50  0001 C CNN
 F 3 "~" H 3900 5600 50  0001 C CNN
 	1    3900 5600
@@
 F 0 "J5" H 3927 5976 50  0000 L CNN
 F 1 "Moisture5" H 3927 5885 50  0000 L CNN
-F 2 "" H 3900 5950 50  0001 C CNN
+F 2 "Connector_PinHeader_2.54mm:PinHeader_1x03_P2.54mm_Vertical" H 3900 5950 50  0001 C CNN
 F 3 "~" H 3900 5950 50  0001 C CNN
 	1    3900 5950
@@
 F 0 "SW1" H 7200 2935 50  0000 C CNN
 F 1 "Reset" H 7200 2844 50  0000 C CNN
-F 2 "" H 7200 2850 50  0001 C CNN
+F 2 "Button_Switch_THT:SW_TH_Tactile_Omron_B3F-10xx" H 7200 2850 50  0001 C CNN
 F 3 "" H 7200 2850 50  0001 C CNN
 	1    7200 2650
@@
 F 0 "R1" H 7570 2446 50  0000 L CNN
 F 1 "10k" H 7570 2355 50  0000 L CNN
-F 2 "" V 7430 2400 50  0001 C CNN
+F 2 "Resistor_THT:R_Axial_DIN0207_L6.3mm_D2.5mm_P10.16mm_Horizontal" V 7430 2400 50  0001 C CNN
 F 3 "~" H 7500 2400 50  0001 C CNN
 	1    7500 2400
@@
 F 0 "R2" H 9120 3746 50  0000 L CNN
 F 1 "10k" H 9120 3655 50  0000 L CNN
-F 2 "" V 8980 3700 50  0001 C CNN
+F 2 "Resistor_THT:R_Axial_DIN0207_L6.3mm_D2.5mm_P10.16mm_Horizontal" V 8980 3700 50  0001 C CNN
 F 3 "~" H 9050 3700 50  0001 C CNN
 	1    9050 3700
@@
 F 0 "R3" H 9470 2246 50  0000 L CNN
 F 1 "10k" H 9470 2155 50  0000 L CNN
-F 2 "" V 9330 2200 50  0001 C CNN
+F 2 "Resistor_THT:R_Axial_DIN0207_L6.3mm_D2.5mm_P10.16mm_Horizontal" V 9330 2200 50  0001 C CNN
 F 3 "~" H 9400 2200 50  0001 C CNN
 	1    9400 2200
@@
 F 0 "SW2" V 9554 2748 50  0000 L CNN
 F 1 "Flash" V 9645 2748 50  0000 L CNN
-F 2 "" H 9600 2800 50  0001 C CNN
+F 2 "Button_Switch_THT:SW_TH_Tactile_Omron_B3F-10xx" H 9600 2800 50  0001 C CNN
 F 3 "" H 9600 2800 50  0001 C CNN
 	1    9600 2600
@@
 F 0 "R4" H 2420 1946 50  0000 L CNN
 F 1 "1.8K" H 2420 1855 50  0000 L CNN
-F 2 "" V 2280 1900 50  0001 C CNN
+F 2 "Resistor_THT:R_Axial_DIN0207_L6.3mm_D2.5mm_P10.16mm_Horizontal" V 2280 1900 50  0001 C CNN
 F 3 "~" H 2350 1900 50  0001 C CNN
 	1    2350 1900
@@
 F 0 "R5" H 2420 2346 50  0000 L CNN
 F 1 "5K" H 2420 2255 50  0000 L CNN
-F 2 "" V 2280 2300 50  0001 C CNN
+F 2 "Resistor_THT:R_Axial_DIN0207_L6.3mm_D2.5mm_P10.16mm_Horizontal" V 2280 2300 50  0001 C CNN
 F 3 "~" H 2350 2300 50  0001 C CNN
 	1    2350 2300
@@
 A5
 $Comp
-L Connector:Screw_Terminal_01x02 J?
+L Connector:Screw_Terminal_01x02 J6
 U 1 1 5D2F0189
 P 650 1200
-F 0 "J?" H 570 875 50  0000 C CNN
+F 0 "J6" H 570 875 50  0000 C CNN
 F 1 "Screw_Terminal_01x02" H 570 966 50  0000 C CNN
-F 2 "" H 650 1200 50  0001 C CNN
+F 2 "TerminalBlock_RND:TerminalBlock_RND_205-00001_1x02_P5.00mm_Horizontal" H 650 1200 50  0001 C CNN
 F 3 "~" H 650 1200 50  0001 C CNN
 	1    650  1200
@@
 Wire Wire Line
 	950  1200 850  1200
-$Comp
-L Connector:Conn_01x03_Female J?
-U 1 1 5D2F4476
-P 8350 5100
-F 0 "J?" H 8377 5126 50  0000 L CNN
-F 1 "Conn_01x03_Female" H 8377 5035 50  0000 L CNN
-F 2 "" H 8350 5100 50  0001 C CNN
-F 3 "~" H 8350 5100 50  0001 C CNN
-	1    8350 5100
-	1    0    0    -1
-$EndComp
 Wire Wire Line
 	8150 5000 8000 5000
@@
 TX
 $Comp
-L power:GND #PWR?
+L power:GND #PWR0101
 U 1 1 5D2FA87B
 P 8000 5200
-F 0 "#PWR?" H 8000 4950 50  0001 C CNN
+F 0 "#PWR0101" H 8000 4950 50  0001 C CNN
 F 1 "GND" H 8005 5027 50  0000 C CNN
 F 2 "" H 8000 5200 50  0001 C CNN
@@
 $EndComp
 $Comp
-L Device:R R?
+L Device:R R6
 U 1 1 5D2FAB4C
 P 6550 1250
-F 0 "R?" H 6620 1296 50  0000 L CNN
+F 0 "R6" H 6620 1296 50  0000 L CNN
 F 1 "R" H 6620 1205 50  0000 L CNN
-F 2 "" V 6480 1250 50  0001 C CNN
+F 2 "Resistor_THT:R_Axial_DIN0207_L6.3mm_D2.5mm_P10.16mm_Horizontal" V 6480 1250 50  0001 C CNN
 F 3 "~" H 6550 1250 50  0001 C CNN
 	1    6550 1250
@@
 Text Label 8850 3050 0    50   ~ 0
 DHT11Data
+$Comp
+L Connector:Conn_01x03_Female J7
+U 1 1 5D2F4476
+P 8350 5100
+F 0 "J7" H 8377 5126 50  0000 L CNN
+F 1 "UART out" H 8377 5035 50  0000 L CNN
+F 2 "Connector_PinHeader_2.54mm:PinHeader_1x03_P2.54mm_Vertical" H 8350 5100 50  0001 C CNN
+F 3 "~" H 8350 5100 50  0001 C CNN
+	1    8350 5100
+	1    0    0    -1
+$EndComp
+$Comp
+L connected_garden_lib:TP4056-18650 U1
+U 1 1 5D383666
+P 1500 1150
+F 0 "U1" H 1475 1625 50  0000 C CNN
+F 1 "TP4056-18650" H 1475 1534 50  0000 C CNN
+F 2 "connected_garden_footprints:TP4056-18650" H 1450 1150 50  0001 C CNN
+F 3 "" H 1450 1150 50  0001 C CNN
+	1    1500 1150
+	1    0    0    -1
+$EndComp
 $EndSCHEMATC

Commit message: Changes MCP3208 footprint, reroute and add text
Parts:
- U2: footprint Package_DIP:DIP-16_W7.62mm_Socket_LongPads -> Package_SO:SOIC-16_3.9x9.9mm_P1.27mm
Changed lines of the file:
@@
 F 0 "U2" H 1700 5828 50  0000 C CNN
 F 1 "MCP3208" H 1700 5737 50  0000 C CNN
-F 2 "Package_DIP:DIP-16_W7.62mm_Socket_LongPads" H 1800 5250 50  0001 C CNN
+F 2 "Package_SO:SOIC-16_3.9x9.9mm_P1.27mm" H 1800 5250 50  0001 C CNN
 F 3 "http://ww1.microchip.com/downloads/en/DeviceDoc/21298c.pdf" H 1800 5250 50  0001 C CNN
 	1    1700 5150

Commit message: [Elec] Adds BUZ11 to shut sensor off
Parts:
- added Q1: BUZ11, Package_TO_SOT_THT:TO-220-3_Vertical, symbol Transistor_FET:BUZ11
- added R7: 220, Resistor_THT:R_Axial_DIN0207_L6.3mm_D2.5mm_P10.16mm_Horizontal, symbol Device:R
- added R8: 10K, Resistor_THT:R_Axial_DIN0207_L6.3mm_D2.5mm_P10.16mm_Horizontal, symbol Device:R
Connections:
- net labels added: 3.3V_EN, GND_EN, MOSG
- wire segments 88 -> 100
Changed lines of the file:
@@
-$EndComp
-$Comp
-L power:GND #PWR013
-U 1 1 5D27D90E
-P 6050 1700
-F 0 "#PWR013" H 6050 1450 50  0001 C CNN
-F 1 "GND" H 6055 1527 50  0000 C CNN
-F 2 "" H 6050 1700 50  0001 C CNN
-F 3 "" H 6050 1700 50  0001 C CNN
-	1    6050 1700
-	1    0    0    -1
-$EndComp
-$Comp
-L power:+3.3V #PWR012
-U 1 1 5D27D940
-P 6050 1100
-F 0 "#PWR012" H 6050 950 50  0001 C CNN
-F 1 "+3.3V" H 6065 1273 50  0000 C CNN
-F 2 "" H 6050 1100 50  0001 C CNN
-F 3 "" H 6050 1100 50  0001 C CNN
-	1    6050 1100
-	1    0    0    -1
 $EndComp
 $Comp
@@
 Wire Wire Line
 	3700 6050 3350 6050
-$Comp
-L power:+3.3V #PWR08
-U 1 1 5D2869C9
-P 3500 4350
-F 0 "#PWR08" H 3500 4200 50  0001 C CNN
-F 1 "+3.3V" H 3515 4523 50  0000 C CNN
-F 2 "" H 3500 4350 50  0001 C CNN
-F 3 "" H 3500 4350 50  0001 C CNN
-	1    3500 4350
-	1    0    0    -1
-$EndComp
-$Comp
-L power:GND #PWR09
-U 1 1 5D286A13
-P 3600 6250
-F 0 "#PWR09" H 3600 6000 50  0001 C CNN
-F 1 "GND" H 3605 6077 50  0000 C CNN
-F 2 "" H 3600 6250 50  0001 C CNN
-F 3 "" H 3600 6250 50  0001 C CNN
-	1    3600 6250
-	1    0    0    -1
-$EndComp
 Text Label 3350 4650 0    50   ~ 0
 A0
@@
 Wire Wire Line
 	6550 1100 6050 1100
-Connection ~ 6050 1100
 Wire Wire Line
 	6550 1400 6450 1400
@@
 	1    0    0    -1
 $EndComp
+Wire Wire Line
+	8750 3250 8850 3250
+$Comp
+L Transistor_FET:BUZ11 Q1
+U 1 1 5D69C850
+P 6400 4950
+F 0 "Q1" H 6606 4996 50  0000 L CNN
+F 1 "BUZ11" H 6606 4905 50  0000 L CNN
+F 2 "Package_TO_SOT_THT:TO-220-3_Vertical" H 6650 4875 50  0001 L CIN
+F 3 "http://www.fairchildsemi.com/ds/BU/BUZ11.pdf" H 6400 4950 50  0001 L CNN
+	1    6400 4950
+	1    0    0    -1
+$EndComp
+Wire Wire Line
+	5950 4950 6100 4950
+Wire Wire Line
+	6100 4950 6100 5050
+Connection ~ 6100 4950
+Wire Wire Line
+	6100 4950 6200 4950
+$Comp
+L Device:R R7
+U 1 1 5D6A3F8B
+P 5800 4950
+F 0 "R7" V 5593 4950 50  0000 C CNN
+F 1 "220" V 5684 4950 50  0000 C CNN
+F 2 "Resistor_THT:R_Axial_DIN0207_L6.3mm_D2.5mm_P10.16mm_Horizontal" V 5730 4950 50  0001 C CNN
+F 3 "~" H 5800 4950 50  0001 C CNN
+	1    5800 4950
+	0    1    1    0
+$EndComp
+$Comp
+L Device:R R8
+U 1 1 5D6A4022
+P 6100 5200
+F 0 "R8" H 6170 5246 50  0000 L CNN
+F 1 "10K" H 6170 5155 50  0000 L CNN
+F 2 "Resistor_THT:R_Axial_DIN0207_L6.3mm_D2.5mm_P10.16mm_Horizontal" V 6030 5200 50  0001 C CNN
+F 3 "~" H 6100 5200 50  0001 C CNN
+	1    6100 5200
+	1    0    0    -1
+$EndComp
+Wire Wire Line
+	6100 5350 6100 5400
+$Comp
+L power:GND #PWR0102
+U 1 1 5D6A69AA
+P 6100 5400
+F 0 "#PWR0102" H 6100 5150 50  0001 C CNN
+F 1 "GND" H 6105 5227 50  0000 C CNN
+F 2 "" H 6100 5400 50  0001 C CNN
+F 3 "" H 6100 5400 50  0001 C CNN
+	1    6100 5400
+	1    0    0    -1
+$EndComp
+$Comp
+L power:GND #PWR0103
+U 1 1 5D6A6B94
+P 6500 5150
+F 0 "#PWR0103" H 6500 4900 50  0001 C CNN
+F 1 "GND" H 6505 4977 50  0000 C CNN
+F 2 "" H 6500 5150 50  0001 C CNN
+F 3 "" H 6500 5150 50  0001 C CNN
+	1    6500 5150
+	1    0    0    -1
+$EndComp
+Wire Wire Line
+	5650 4950 5550 4950
+Wire Wire Line
+	6500 4750 6500 4600
+Wire Wire Line
+	6500 4600 6600 4600
+Wire Wire Line
+	6600 4450 6500 4450
+Wire Wire Line
+	6500 4450 6500 4350
+$Comp
+L power:+3.3V #PWR0104
+U 1 1 5D6B17B3
+P 6500 4350
+F 0 "#PWR0104" H 6500 4200 50  0001 C CNN
+F 1 "+3.3V" H 6515 4523 50  0000 C CNN
+F 2 "" H 6500 4350 50  0001 C CNN
+F 3 "" H 6500 4350 50  0001 C CNN
+	1    6500 4350
+	1    0    0    -1
+$EndComp
+Text Label 6600 4450 0    50   ~ 0
+3.3V_EN
+Text Label 6600 4600 0    50   ~ 0
+GND_EN
+Text Label 5550 4950 0    50   ~ 0
+MOSG
+Text Label 8850 3250 0    50   ~ 0
+MOSG
+Wire Wire Line
+	6050 1100 6050 1000
+Connection ~ 6050 1100
+Text Label 6050 1000 0    50   ~ 0
+3.3V_EN
+Wire Wire Line
+	6050 1700 6050 1800
+Text Label 6050 1800 0    50   ~ 0
+GND_EN
+Text Label 3500 4350 0    50   ~ 0
+3.3V_EN
+Text Label 3600 6250 0    50   ~ 0
+GND_EN
 $EndSCHEMATC
